Commit message: feat: add primitive geometry visuals to example URDF xacros
Each example now has full visual/collision/inertial blocks using standard
shapes (no external mesh files required), so robot_state_publisher +
RViz2/Foxglove will render something immediately:

single_motor_position.urdf.xacro:
  - base_link: 80×80×5 mm grey box (mounting plate)
  - arm_link:  40×20×40 mm dark-grey box (STS3215 body, origin at shaft)
               + 50×8×8 mm orange box (servo horn / arm extending +x)

single_motor_velocity.urdf.xacro:
  - base_link: 100×100×5 mm grey box
  - wheel_link: r=30 mm blue cylinder (drive wheel, axis Z)
                + 40×40×20 mm dark-grey box (servo body behind wheel)

mixed_mode.urdf.xacro:
  - base_link: 100×100×5 mm grey box
  - arm_link_1/2: STS3215 body + orange horn (same as position example)
  - wheel_link_1/2: blue wheel cylinder + dark-grey servo body
  - gripper_link_1/2: 60×10×8 mm green box (finger, origin at root)
  Joint origins updated to place children at realistic positions.

File: config/mixed_mode.urdf.xacro (robot description, xacro)
@@ -6,19 +6,197 @@
   <xacro:arg name="use_mock" default="false"/>
   <!-- Robot description -->
-  <link name="base_link"/>
-  <!-- Position Mode Links (Mode 0) -->
-  <link name="arm_link_1"/>
-  <link name="arm_link_2"/>
-  <!-- Velocity Mode Links (Mode 1) -->
-  <link name="wheel_link_1"/>
-  <link name="wheel_link_2"/>
-  <!-- PWM Mode Links (Mode 2) -->
-  <link name="gripper_link_1"/>
-  <link name="gripper_link_2"/>
+  <!-- base_link: flat mounting plate (100×100×5 mm) -->
+  <link name="base_link">
+    <visual>
+      <geometry>
+        <box size="0.10 0.10 0.005"/>
+      </geometry>
+      <material name="grey">
+        <color rgba="0.5 0.5 0.5 1.0"/>
+      </material>
+    </visual>
+    <collision>
+      <geometry>
+        <box size="0.10 0.10 0.005"/>
+      </geometry>
+    </collision>
+    <inertial>
+      <mass value="0.05"/>
+      <inertia ixx="0.00004" ixy="0" ixz="0" iyy="0.00004" iyz="0" izz="0.00008"/>
+    </inertial>
+  </link>
+  <!-- ─── Position Mode Links (Mode 0) ─── -->
+  <!-- arm_link_1/2: STS3215 servo body + horn extending along +x -->
+  <link name="arm_link_1">
+    <visual>
+      <origin xyz="0 0 -0.02" rpy="0 0 0"/>
+      <geometry>
+        <box size="0.040 0.020 0.040"/>
+      </geometry>
+      <material name="dark_grey">
+        <color rgba="0.2 0.2 0.2 1.0"/>
+      </material>
+    </visual>
+    <visual>
+      <origin xyz="0.035 0 0" rpy="0 0 0"/>
+      <geometry>
+        <box size="0.05 0.008 0.008"/>
+      </geometry>
+      <material name="orange">
+        <color rgba="1.0 0.5 0.0 1.0"/>
+      </material>
+    </visual>
+    <collision>
+      <origin xyz="0 0 -0.02" rpy="0 0 0"/>
+      <geometry>
+        <box size="0.040 0.020 0.040"/>
+      </geometry>
+    </collision>
+    <inertial>
+      <mass value="0.068"/>
+      <origin xyz="0 0 -0.02"/>
+      <inertia ixx="0.000015" ixy="0" ixz="0" iyy="0.000015" iyz="0" izz="0.000007"/>
+    </inertial>
+  </link>
+  <link name="arm_link_2">
+    <visual>
+      <origin xyz="0 0 -0.02" rpy="0 0 0"/>
+      <geometry>
+        <box size="0.040 0.020 0.040"/>
+      </geometry>
+      <material name="dark_grey">
+        <color rgba="0.2 0.2 0.2 1.0"/>
+      </material>
+    </visual>
+    <visual>
+      <origin xyz="0.035 0 0" rpy="0 0 0"/>
+      <geometry>
+        <box size="0.05 0.008 0.008"/>
+      </geometry>
+      <material name="orange">
+        <color rgba="1.0 0.5 0.0 1.0"/>
+      </material>
+    </visual>
+    <collision>
+      <origin xyz="0 0 -0.02" rpy="0 0 0"/>
+      <geometry>
+        <box size="0.040 0.020 0.040"/>
+      </geometry>
+    </collision>
+    <inertial>
+      <mass value="0.068"/>
+      <origin xyz="0 0 -0.02"/>
+      <inertia ixx="0.000015" ixy="0" ixz="0" iyy="0.000015" iyz="0" izz="0.000007"/>
+    </inertial>
+  </link>
+  <!-- ─── Velocity Mode Links (Mode 1) ─── -->
+  <!-- wheel_link_1/2: cylinder (r=30 mm, h=10 mm) + servo body behind -->
+  <link name="wheel_link_1">
+    <visual>
+      <geometry>
+        <cylinder radius="0.030" length="0.010"/>
+      </geometry>
+      <material name="blue">
+        <color rgba="0.1 0.4 0.8 1.0"/>
+      </material>
+    </visual>
+    <visual>
+      <origin xyz="0 -0.025 0" rpy="1.5708 0 0"/>
+      <geometry>
+        <box size="0.040 0.040 0.020"/>
+      </geometry>
+      <material name="dark_grey">
+        <color rgba="0.2 0.2 0.2 1.0"/>
+      </material>
+    </visual>
+    <collision>
+      <geometry>
+        <cylinder radius="0.030" length="0.010"/>
+      </geometry>
+    </collision>
+    <inertial>
+      <mass value="0.068"/>
+      <inertia ixx="0.000015" ixy="0" ixz="0" iyy="0.000015" iyz="0" izz="0.000029"/>
+    </inertial>
+  </link>
+  <link name="wheel_link_2">
+    <visual>
+      <geometry>
+        <cylinder radius="0.030" length="0.010"/>
+      </geometry>
+      <material name="blue">
+        <color rgba="0.1 0.4 0.8 1.0"/>
+      </material>
+    </visual>
+    <visual>
+      <origin xyz="0 0.025 0" rpy="1.5708 0 0"/>
+      <geometry>
+        <box size="0.040 0.040 0.020"/>
+      </geometry>
+      <material name="dark_grey">
+        <color rgba="0.2 0.2 0.2 1.0"/>
+      </material>
+    </visual>
+    <collision>
+      <geometry>
+        <cylinder radius="0.030" length="0.010"/>
+      </geometry>
+    </collision>
+    <inertial>
+      <mass value="0.068"/>
+      <inertia ixx="0.000015" ixy="0" ixz="0" iyy="0.000015" iyz="0" izz="0.000029"/>
+    </inertial>
+  </link>
+  <!-- ─── PWM Mode Links (Mode 2) ─── -->
+  <!-- gripper_link_1/2: thin flat finger -->
+  <link name="gripper_link_1">
+    <visual>
+      <origin xyz="0.03 0 0" rpy="0 0 0"/>
+      <geometry>
+        <box size="0.060 0.010 0.008"/>
+      </geometry>
+      <material name="green">
+        <color rgba="0.1 0.7 0.2 1.0"/>
+      </material>
+    </visual>
+    <collision>
+      <origin xyz="0.03 0 0" rpy="0 0 0"/>
+      <geometry>
+        <box size="0.060 0.010 0.008"/>
+      </geometry>
+    </collision>
+    <inertial>
+      <mass value="0.010"/>
+      <origin xyz="0.03 0 0"/>
+      <inertia ixx="0.0000001" ixy="0" ixz="0" iyy="0.0000030" iyz="0" izz="0.0000030"/>
+    </inertial>
+  </link>
+  <link name="gripper_link_2">
+    <visual>
+      <origin xyz="0.03 0 0" rpy="0 0 0"/>
+      <geometry>
+        <box size="0.060 0.010 0.008"/>
+      </geometry>
+      <material name="green">
+        <color rgba="0.1 0.7 0.2 1.0"/>
+      </material>
+    </visual>
+    <collision>
+      <origin xyz="0.03 0 0" rpy="0 0 0"/>
+      <geometry>
+        <box size="0.060 0.010 0.008"/>
+      </geometry>
+    </collision>
+    <inertial>
+      <mass value="0.010"/>
+      <origin xyz="0.03 0 0"/>
+      <inertia ixx="0.0000001" ixy="0" ixz="0" iyy="0.0000030" iyz="0" izz="0.0000030"/>
+    </inertial>
+  </link>
   <!-- Position Mode Joints (Mode 0) - IDs 1 and 2 -->
   <joint name="arm_joint_1" type="revolute">
     <parent link="base_link"/>
     <child link="arm_link_1"/>
-    <origin xyz="0 0.05 0.1" rpy="0 0 0"/>
+    <origin xyz="0 0.05 0.02" rpy="0 0 0"/>
     <axis xyz="0 1 0"/>
     <limit lower="0.0" upper="6.283" effort="1.0" velocity="5.0"/>
@@ -27,5 +205,5 @@
     <parent link="base_link"/>
     <child link="arm_link_2"/>
-    <origin xyz="0 -0.05 0.1" rpy="0 0 0"/>
+    <origin xyz="0 -0.05 0.02" rpy="0 0 0"/>
     <axis xyz="0 1 0"/>
     <limit lower="0.0" upper="6.283" effort="1.0" velocity="5.0"/>
@@ -35,5 +213,5 @@
     <parent link="base_link"/>
     <child link="wheel_link_1"/>
-    <origin xyz="0.1 0 0" rpy="0 0 0"/>
+    <origin xyz="0.1 0 0.035" rpy="0 0 0"/>
     <axis xyz="0 0 1"/>
   </joint>
@@ -41,5 +219,5 @@
     <parent link="base_link"/>
     <child link="wheel_link_2"/>
-    <origin xyz="-0.1 0 0" rpy="0 0 0"/>
+    <origin xyz="-0.1 0 0.035" rpy="0 0 0"/>
     <axis xyz="0 0 1"/>
   </joint>
@@ -48,5 +226,5 @@
     <parent link="arm_link_1"/>
     <child link="gripper_link_1"/>
-    <origin xyz="0.2 0 0" rpy="0 0 0"/>
+    <origin xyz="0.06 0 0" rpy="0 0 0"/>
     <axis xyz="0 0 1"/>
     <limit lower="0.0" upper="0.5" effort="1.0" velocity="2.0"/>
@@ -55,5 +233,5 @@
     <parent link="arm_link_2"/>
     <child link="gripper_link_2"/>
-    <origin xyz="0.2 0 0" rpy="0 0 0"/>
+    <origin xyz="0.06 0 0" rpy="0 0 0"/>
     <axis xyz="0 0 1"/>
     <limit lower="0.0" upper="0.5" effort="1.0" velocity="2.0"/>

File: config/single_motor_position.urdf.xacro (robot description, xacro)
@@ -7,10 +7,63 @@
   <xacro:arg name="use_mock" default="false"/>
   <!-- Robot description -->
-  <link name="base_link"/>
-  <link name="arm_link"/>
+  <!-- base_link: flat mounting plate -->
+  <link name="base_link">
+    <visual>
+      <geometry>
+        <box size="0.08 0.08 0.005"/>
+      </geometry>
+      <material name="grey">
+        <color rgba="0.5 0.5 0.5 1.0"/>
+      </material>
+    </visual>
+    <collision>
+      <geometry>
+        <box size="0.08 0.08 0.005"/>
+      </geometry>
+    </collision>
+    <inertial>
+      <mass value="0.05"/>
+      <inertia ixx="0.00003" ixy="0" ixz="0" iyy="0.00003" iyz="0" izz="0.00005"/>
+    </inertial>
+  </link>
+  <!-- STS3215 servo body: 40×20×40 mm box, joint origin sits at the output shaft centre -->
+  <link name="arm_link">
+    <visual>
+      <!-- servo body: 40mm wide (x), 20mm deep (y), 40mm tall (z); shaft at top centre -->
+      <origin xyz="0 0 -0.02" rpy="0 0 0"/>
+      <geometry>
+        <box size="0.040 0.020 0.040"/>
+      </geometry>
+      <material name="dark_grey">
+        <color rgba="0.2 0.2 0.2 1.0"/>
+      </material>
+    </visual>
+    <!-- servo horn: thin flat arm extending +x from shaft -->
+    <visual>
+      <origin xyz="0.035 0 0" rpy="0 0 0"/>
+      <geometry>
+        <box size="0.05 0.008 0.008"/>
+      </geometry>
+      <material name="orange">
+        <color rgba="1.0 0.5 0.0 1.0"/>
+      </material>
+    </visual>
+    <collision>
+      <origin xyz="0 0 -0.02" rpy="0 0 0"/>
+      <geometry>
+        <box size="0.040 0.020 0.040"/>
+      </geometry>
+    </collision>
+    <inertial>
+      <mass value="0.068"/>
+      <origin xyz="0 0 -0.02"/>
+      <inertia ixx="0.000015" ixy="0" ixz="0" iyy="0.000015" iyz="0" izz="0.000007"/>
+    </inertial>
+  </link>
   <joint name="arm_joint" type="revolute">
     <parent link="base_link"/>
     <child link="arm_link"/>
-    <origin xyz="0 0 0" rpy="0 0 0"/>
+    <!-- shaft sits 20 mm above the base plate -->
+    <origin xyz="0 0 0.02" rpy="0 0 0"/>
     <axis xyz="0 1 0"/>
     <limit lower="0.0" upper="6.283" effort="1.0" velocity="5.0"/>

File: config/single_motor_velocity.urdf.xacro (robot description, xacro)
@@ -7,10 +7,61 @@
   <xacro:arg name="use_mock" default="false"/>
   <!-- Robot description -->
-  <link name="base_link"/>
-  <link name="wheel_link"/>
+  <!-- base_link: flat mounting plate -->
+  <link name="base_link">
+    <visual>
+      <geometry>
+        <box size="0.10 0.10 0.005"/>
+      </geometry>
+      <material name="grey">
+        <color rgba="0.5 0.5 0.5 1.0"/>
+      </material>
+    </visual>
+    <collision>
+      <geometry>
+        <box size="0.10 0.10 0.005"/>
+      </geometry>
+    </collision>
+    <inertial>
+      <mass value="0.05"/>
+      <inertia ixx="0.00004" ixy="0" ixz="0" iyy="0.00004" iyz="0" izz="0.00008"/>
+    </inertial>
+  </link>
+  <!-- wheel_link: cylinder representing a drive wheel, shaft along Z -->
+  <link name="wheel_link">
+    <visual>
+      <!-- wheel disc -->
+      <origin xyz="0 0 0" rpy="0 0 0"/>
+      <geometry>
+        <cylinder radius="0.030" length="0.010"/>
+      </geometry>
+      <material name="blue">
+        <color rgba="0.1 0.4 0.8 1.0"/>
+      </material>
+    </visual>
+    <!-- STS3215 servo body behind the wheel -->
+    <visual>
+      <origin xyz="0 -0.025 0" rpy="1.5708 0 0"/>
+      <geometry>
+        <box size="0.040 0.040 0.020"/>
+      </geometry>
+      <material name="dark_grey">
+        <color rgba="0.2 0.2 0.2 1.0"/>
+      </material>
+    </visual>
+    <collision>
+      <geometry>
+        <cylinder radius="0.030" length="0.010"/>
+      </geometry>
+    </collision>
+    <inertial>
+      <mass value="0.068"/>
+      <inertia ixx="0.000015" ixy="0" ixz="0" iyy="0.000015" iyz="0" izz="0.000029"/>
+    </inertial>
+  </link>
   <joint name="wheel_joint" type="continuous">
     <parent link="base_link"/>
     <child link="wheel_link"/>
-    <origin xyz="0 0 0" rpy="0 0 0"/>
+    <!-- wheel shaft 35 mm above the plate, centred -->
+    <origin xyz="0 0 0.035" rpy="0 0 0"/>
     <axis xyz="0 0 1"/>
   </joint>
