Commit message: chore: remove primitive geometry from example URDF xacros
Reverts the visual/collision/inertial geometry blocks added in 2c620e7.
Example xacros are reference configurations for the hardware interface
parameters, not robot visualisation files — empty links are clearer and
avoid KDL/inertia warnings from robot_state_publisher.

All four files restored to bare-link + joint structure:
- single_motor_position.urdf.xacro
- single_motor_velocity.urdf.xacro
- single_motor_pwm.urdf.xacro  (continuous joint retained from 7a2474b)
- mixed_mode.urdf.xacro         (joint origins restored to original values)

Also fixes a duplicate '<!-- Robot description -->' comment in
single_motor_pwm.urdf.xacro left from the geometry removal.

File: config/mixed_mode.urdf.xacro (robot description, xacro)
@@ -6,197 +6,19 @@
   <xacro:arg name="use_mock" default="false"/>
   <!-- Robot description -->
-  <!-- base_link: flat mounting plate (100×100×5 mm) -->
-  <link name="base_link">
-    <visual>
-      <geometry>
-        <box size="0.10 0.10 0.005"/>
-      </geometry>
-      <material name="grey">
-        <color rgba="0.5 0.5 0.5 1.0"/>
-      </material>
-    </visual>
-    <collision>
-      <geometry>
-        <box size="0.10 0.10 0.005"/>
-      </geometry>
-    </collision>
-    <inertial>
-      <mass value="0.05"/>
-      <inertia ixx="0.00004" ixy="0" ixz="0" iyy="0.00004" iyz="0" izz="0.00008"/>
-    </inertial>
-  </link>
-  <!-- ─── Position Mode Links (Mode 0) ─── -->
-  <!-- arm_link_1/2: STS3215 servo body + horn extending along +x -->
-  <link name="arm_link_1">
-    <visual>
-      <origin xyz="0 0 -0.02" rpy="0 0 0"/>
-      <geometry>
-        <box size="0.040 0.020 0.040"/>
-      </geometry>
-      <material name="dark_grey">
-        <color rgba="0.2 0.2 0.2 1.0"/>
-      </material>
-    </visual>
-    <visual>
-      <origin xyz="0.035 0 0" rpy="0 0 0"/>
-      <geometry>
-        <box size="0.05 0.008 0.008"/>
-      </geometry>
-      <material name="orange">
-        <color rgba="1.0 0.5 0.0 1.0"/>
-      </material>
-    </visual>
-    <collision>
-      <origin xyz="0 0 -0.02" rpy="0 0 0"/>
-      <geometry>
-        <box size="0.040 0.020 0.040"/>
-      </geometry>
-    </collision>
-    <inertial>
-      <mass value="0.068"/>
-      <origin xyz="0 0 -0.02"/>
-      <inertia ixx="0.000015" ixy="0" ixz="0" iyy="0.000015" iyz="0" izz="0.000007"/>
-    </inertial>
-  </link>
-  <link name="arm_link_2">
-    <visual>
-      <origin xyz="0 0 -0.02" rpy="0 0 0"/>
-      <geometry>
-        <box size="0.040 0.020 0.040"/>
-      </geometry>
-      <material name="dark_grey">
-        <color rgba="0.2 0.2 0.2 1.0"/>
-      </material>
-    </visual>
-    <visual>
-      <origin xyz="0.035 0 0" rpy="0 0 0"/>
-      <geometry>
-        <box size="0.05 0.008 0.008"/>
-      </geometry>
-      <material name="orange">
-        <color rgba="1.0 0.5 0.0 1.0"/>
-      </material>
-    </visual>
-    <collision>
-      <origin xyz="0 0 -0.02" rpy="0 0 0"/>
-      <geometry>
-        <box size="0.040 0.020 0.040"/>
-      </geometry>
-    </collision>
-    <inertial>
-      <mass value="0.068"/>
-      <origin xyz="0 0 -0.02"/>
-      <inertia ixx="0.000015" ixy="0" ixz="0" iyy="0.000015" iyz="0" izz="0.000007"/>
-    </inertial>
-  </link>
-  <!-- ─── Velocity Mode Links (Mode 1) ─── -->
-  <!-- wheel_link_1/2: cylinder (r=30 mm, h=10 mm) + servo body behind -->
-  <link name="wheel_link_1">
-    <visual>
-      <geometry>
-        <cylinder radius="0.030" length="0.010"/>
-      </geometry>
-      <material name="blue">
-        <color rgba="0.1 0.4 0.8 1.0"/>
-      </material>
-    </visual>
-    <visual>
-      <origin xyz="0 -0.025 0" rpy="1.5708 0 0"/>
-      <geometry>
-        <box size="0.040 0.040 0.020"/>
-      </geometry>
-      <material name="dark_grey">
-        <color rgba="0.2 0.2 0.2 1.0"/>
-      </material>
-    </visual>
-    <collision>
-      <geometry>
-        <cylinder radius="0.030" length="0.010"/>
-      </geometry>
-    </collision>
-    <inertial>
-      <mass value="0.068"/>
-      <inertia ixx="0.000015" ixy="0" ixz="0" iyy="0.000015" iyz="0" izz="0.000029"/>
-    </inertial>
-  </link>
-  <link name="wheel_link_2">
-    <visual>
-      <geometry>
-        <cylinder radius="0.030" length="0.010"/>
-      </geometry>
-      <material name="blue">
-        <color rgba="0.1 0.4 0.8 1.0"/>
-      </material>
-    </visual>
-    <visual>
-      <origin xyz="0 0.025 0" rpy="1.5708 0 0"/>
-      <geometry>
-        <box size="0.040 0.040 0.020"/>
-      </geometry>
-      <material name="dark_grey">
-        <color rgba="0.2 0.2 0.2 1.0"/>
-      </material>
-    </visual>
-    <collision>
-      <geometry>
-        <cylinder radius="0.030" length="0.010"/>
-      </geometry>
-    </collision>
-    <inertial>
-      <mass value="0.068"/>
-      <inertia ixx="0.000015" ixy="0" ixz="0" iyy="0.000015" iyz="0" izz="0.000029"/>
-    </inertial>
-  </link>
-  <!-- ─── PWM Mode Links (Mode 2) ─── -->
-  <!-- gripper_link_1/2: thin flat finger -->
-  <link name="gripper_link_1">
-    <visual>
-      <origin xyz="0.03 0 0" rpy="0 0 0"/>
-      <geometry>
-        <box size="0.060 0.010 0.008"/>
-      </geometry>
-      <material name="green">
-        <color rgba="0.1 0.7 0.2 1.0"/>
-      </material>
-    </visual>
-    <collision>
-      <origin xyz="0.03 0 0" rpy="0 0 0"/>
-      <geometry>
-        <box size="0.060 0.010 0.008"/>
-      </geometry>
-    </collision>
-    <inertial>
-      <mass value="0.010"/>
-      <origin xyz="0.03 0 0"/>
-      <inertia ixx="0.0000001" ixy="0" ixz="0" iyy="0.0000030" iyz="0" izz="0.0000030"/>
-    </inertial>
-  </link>
-  <link name="gripper_link_2">
-    <visual>
-      <origin xyz="0.03 0 0" rpy="0 0 0"/>
-      <geometry>
-        <box size="0.060 0.010 0.008"/>
-      </geometry>
-      <material name="green">
-        <color rgba="0.1 0.7 0.2 1.0"/>
-      </material>
-    </visual>
-    <collision>
-      <origin xyz="0.03 0 0" rpy="0 0 0"/>
-      <geometry>
-        <box size="0.060 0.010 0.008"/>
-      </geometry>
-    </collision>
-    <inertial>
-      <mass value="0.010"/>
-      <origin xyz="0.03 0 0"/>
-      <inertia ixx="0.0000001" ixy="0" ixz="0" iyy="0.0000030" iyz="0" izz="0.0000030"/>
-    </inertial>
-  </link>
+  <!-- Position Mode Links (Mode 0) -->
+  <link name="base_link"/>
+  <link name="arm_link_1"/>
+  <link name="arm_link_2"/>
+  <!-- Velocity Mode Links (Mode 1) -->
+  <link name="wheel_link_1"/>
+  <link name="wheel_link_2"/>
+  <!-- PWM Mode Links (Mode 2) -->
+  <link name="gripper_link_1"/>
+  <link name="gripper_link_2"/>
   <!-- Position Mode Joints (Mode 0) - IDs 1 and 2 -->
   <joint name="arm_joint_1" type="revolute">
     <parent link="base_link"/>
     <child link="arm_link_1"/>
-    <origin xyz="0 0.05 0.02" rpy="0 0 0"/>
+    <origin xyz="0 0.05 0.1" rpy="0 0 0"/>
     <axis xyz="0 1 0"/>
     <limit lower="0.0" upper="6.283" effort="1.0" velocity="5.0"/>
@@ -205,5 +27,5 @@
     <parent link="base_link"/>
     <child link="arm_link_2"/>
-    <origin xyz="0 -0.05 0.02" rpy="0 0 0"/>
+    <origin xyz="0 -0.05 0.1" rpy="0 0 0"/>
     <axis xyz="0 1 0"/>
     <limit lower="0.0" upper="6.283" effort="1.0" velocity="5.0"/>
@@ -213,5 +35,5 @@
     <parent link="base_link"/>
     <child link="wheel_link_1"/>
-    <origin xyz="0.1 0 0.035" rpy="0 0 0"/>
+    <origin xyz="0.1 0 0" rpy="0 0 0"/>
     <axis xyz="0 0 1"/>
   </joint>
@@ -219,5 +41,5 @@
     <parent link="base_link"/>
     <child link="wheel_link_2"/>
-    <origin xyz="-0.1 0 0.035" rpy="0 0 0"/>
+    <origin xyz="-0.1 0 0" rpy="0 0 0"/>
     <axis xyz="0 0 1"/>
   </joint>
@@ -226,5 +48,5 @@
     <parent link="arm_link_1"/>
     <child link="gripper_link_1"/>
-    <origin xyz="0.06 0 0" rpy="0 0 0"/>
+    <origin xyz="0.2 0 0" rpy="0 0 0"/>
     <axis xyz="0 0 1"/>
     <limit lower="0.0" upper="0.5" effort="1.0" velocity="2.0"/>
@@ -233,5 +55,5 @@
     <parent link="arm_link_2"/>
     <child link="gripper_link_2"/>
-    <origin xyz="0.06 0 0" rpy="0 0 0"/>
+    <origin xyz="0.2 0 0" rpy="0 0 0"/>
     <axis xyz="0 0 1"/>
     <limit lower="0.0" upper="0.5" effort="1.0" velocity="2.0"/>

File: config/single_motor_position.urdf.xacro (robot description, xacro)
@@ -7,63 +7,10 @@
   <xacro:arg name="use_mock" default="false"/>
   <!-- Robot description -->
-  <!-- base_link: flat mounting plate -->
-  <link name="base_link">
-    <visual>
-      <geometry>
-        <box size="0.08 0.08 0.005"/>
-      </geometry>
-      <material name="grey">
-        <color rgba="0.5 0.5 0.5 1.0"/>
-      </material>
-    </visual>
-    <collision>
-      <geometry>
-        <box size="0.08 0.08 0.005"/>
-      </geometry>
-    </collision>
-    <inertial>
-      <mass value="0.05"/>
-      <inertia ixx="0.00003" ixy="0" ixz="0" iyy="0.00003" iyz="0" izz="0.00005"/>
-    </inertial>
-  </link>
-  <!-- STS3215 servo body: 40×20×40 mm box, joint origin sits at the output shaft centre -->
-  <link name="arm_link">
-    <visual>
-      <!-- servo body: 40mm wide (x), 20mm deep (y), 40mm tall (z); shaft at top centre -->
-      <origin xyz="0 0 -0.02" rpy="0 0 0"/>
-      <geometry>
-        <box size="0.040 0.020 0.040"/>
-      </geometry>
-      <material name="dark_grey">
-        <color rgba="0.2 0.2 0.2 1.0"/>
-      </material>
-    </visual>
-    <!-- servo horn: thin flat arm extending +x from shaft -->
-    <visual>
-      <origin xyz="0.035 0 0" rpy="0 0 0"/>
-      <geometry>
-        <box size="0.05 0.008 0.008"/>
-      </geometry>
-      <material name="orange">
-        <color rgba="1.0 0.5 0.0 1.0"/>
-      </material>
-    </visual>
-    <collision>
-      <origin xyz="0 0 -0.02" rpy="0 0 0"/>
-      <geometry>
-        <box size="0.040 0.020 0.040"/>
-      </geometry>
-    </collision>
-    <inertial>
-      <mass value="0.068"/>
-      <origin xyz="0 0 -0.02"/>
-      <inertia ixx="0.000015" ixy="0" ixz="0" iyy="0.000015" iyz="0" izz="0.000007"/>
-    </inertial>
-  </link>
+  <link name="base_link"/>
+  <link name="arm_link"/>
   <joint name="arm_joint" type="revolute">
     <parent link="base_link"/>
     <child link="arm_link"/>
-    <!-- shaft sits 20 mm above the base plate -->
-    <origin xyz="0 0 0.02" rpy="0 0 0"/>
+    <origin xyz="0 0 0" rpy="0 0 0"/>
     <axis xyz="0 1 0"/>
     <limit lower="0.0" upper="6.283" effort="1.0" velocity="5.0"/>

File: config/single_motor_pwm.urdf.xacro (robot description, xacro)
@@ -8,67 +8,9 @@
   <xacro:arg name="max_effort" default="1.0"/>
   <!-- Robot description -->
-  <!-- base_link: flat mounting plate -->
-  <link name="base_link">
-    <visual>
-      <geometry>
-        <box size="0.08 0.08 0.005"/>
-      </geometry>
-      <material name="grey">
-        <color rgba="0.5 0.5 0.5 1.0"/>
-      </material>
-    </visual>
-    <collision>
-      <geometry>
-        <box size="0.08 0.08 0.005"/>
-      </geometry>
-    </collision>
-    <inertial>
-      <mass value="0.05"/>
-      <inertia ixx="0.00003" ixy="0" ixz="0" iyy="0.00003" iyz="0" izz="0.00005"/>
-    </inertial>
-  </link>
-  <!-- pwm_link: STS3215 servo body (40×20×40 mm) + output horn extending +x.
-       In Mode 2 the motor is open-loop; the horn position is driven directly by
-       PWM duty cycle, so no position feedback loop is active.  The visual still
-       shows the servo body centred on the output shaft (origin). -->
-  <link name="pwm_link">
-    <visual>
-      <!-- servo body: shaft at top-centre, body hangs 20 mm below -->
-      <origin xyz="0 0 -0.02" rpy="0 0 0"/>
-      <geometry>
-        <box size="0.040 0.020 0.040"/>
-      </geometry>
-      <material name="dark_grey">
-        <color rgba="0.2 0.2 0.2 1.0"/>
-      </material>
-    </visual>
-    <!-- output horn: thin arm extending +x from shaft -->
-    <visual>
-      <origin xyz="0.035 0 0" rpy="0 0 0"/>
-      <geometry>
-        <box size="0.05 0.008 0.008"/>
-      </geometry>
-      <material name="red">
-        <!-- red distinguishes this from position-mode orange to make the mode
-             obvious at a glance in RViz2/Foxglove -->
-        <color rgba="0.9 0.1 0.1 1.0"/>
-      </material>
-    </visual>
-    <collision>
-      <origin xyz="0 0 -0.02" rpy="0 0 0"/>
-      <geometry>
-        <box size="0.040 0.020 0.040"/>
-      </geometry>
-    </collision>
-    <inertial>
-      <mass value="0.068"/>
-      <origin xyz="0 0 -0.02"/>
-      <inertia ixx="0.000015" ixy="0" ixz="0" iyy="0.000015" iyz="0" izz="0.000007"/>
-    </inertial>
-  </link>
-  <!-- continuous: PWM mode is open-loop — no position limits apply, the motor
-       runs at the commanded duty cycle indefinitely in either direction.
-       Using continuous avoids JointSaturationLimiter clamping effort to 0
-       when the joint reaches a revolute position limit. -->
+  <!-- Robot description -->
+  <link name="base_link"/>
+  <link name="pwm_link"/>
+  <!-- continuous: PWM mode is open-loop — no position limits apply.
+       Using continuous avoids JointSaturationLimiter clamping effort to 0. -->
   <joint name="pwm_joint" type="continuous">
     <parent link="base_link"/>

File: config/single_motor_velocity.urdf.xacro (robot description, xacro)
@@ -7,61 +7,10 @@
   <xacro:arg name="use_mock" default="false"/>
   <!-- Robot description -->
-  <!-- base_link: flat mounting plate -->
-  <link name="base_link">
-    <visual>
-      <geometry>
-        <box size="0.10 0.10 0.005"/>
-      </geometry>
-      <material name="grey">
-        <color rgba="0.5 0.5 0.5 1.0"/>
-      </material>
-    </visual>
-    <collision>
-      <geometry>
-        <box size="0.10 0.10 0.005"/>
-      </geometry>
-    </collision>
-    <inertial>
-      <mass value="0.05"/>
-      <inertia ixx="0.00004" ixy="0" ixz="0" iyy="0.00004" iyz="0" izz="0.00008"/>
-    </inertial>
-  </link>
-  <!-- wheel_link: cylinder representing a drive wheel, shaft along Z -->
-  <link name="wheel_link">
-    <visual>
-      <!-- wheel disc -->
-      <origin xyz="0 0 0" rpy="0 0 0"/>
-      <geometry>
-        <cylinder radius="0.030" length="0.010"/>
-      </geometry>
-      <material name="blue">
-        <color rgba="0.1 0.4 0.8 1.0"/>
-      </material>
-    </visual>
-    <!-- STS3215 servo body behind the wheel -->
-    <visual>
-      <origin xyz="0 -0.025 0" rpy="1.5708 0 0"/>
-      <geometry>
-        <box size="0.040 0.040 0.020"/>
-      </geometry>
-      <material name="dark_grey">
-        <color rgba="0.2 0.2 0.2 1.0"/>
-      </material>
-    </visual>
-    <collision>
-      <geometry>
-        <cylinder radius="0.030" length="0.010"/>
-      </geometry>
-    </collision>
-    <inertial>
-      <mass value="0.068"/>
-      <inertia ixx="0.000015" ixy="0" ixz="0" iyy="0.000015" iyz="0" izz="0.000029"/>
-    </inertial>
-  </link>
+  <link name="base_link"/>
+  <link name="wheel_link"/>
   <joint name="wheel_joint" type="continuous">
     <parent link="base_link"/>
     <child link="wheel_link"/>
-    <!-- wheel shaft 35 mm above the plate, centred -->
-    <origin xyz="0 0 0.035" rpy="0 0 0"/>
+    <origin xyz="0 0 0" rpy="0 0 0"/>
     <axis xyz="0 0 1"/>
   </joint>
