Commit message: fix: use continuous joint and minimal yaml for PWM example
Two fixes found during mock-mode testing:

1. single_motor_pwm.urdf.xacro: change pwm_joint from revolute to
   continuous. Revolute joints have position limits; JointSaturationLimiter
   clamped effort to 0.0 once position hit the upper limit (π rad after
   ~3s at 5 rad/s). PWM mode is open-loop — no position limits apply.

2. single_motor_pwm_controllers.yaml: remove unsupported
   command_interfaces/state_interfaces keys from pwm_controller block.
   JointGroupEffortController does not accept these parameters and they
   were preventing the controller from properly claiming the effort
   command interface (effort stayed 0.0 despite commands being received).

Verified in mock mode:
  effort=0.5 → velocity=5.0, effort≈0.96, is_moving=1.0 ✓
  temperature/current/voltage simulate load correctly ✓
  position accumulates freely past ±π without clamping ✓

File: config/single_motor_pwm.urdf.xacro (robot description, xacro)
@@ -67,7 +67,9 @@
     </inertial>
   </link>
-  <!-- revolute so the horn visually sweeps when effort commands drive it;
-       limits are intentionally wide — PWM mode has no closed-loop position cap -->
-  <joint name="pwm_joint" type="revolute">
+  <!-- continuous: PWM mode is open-loop — no position limits apply, the motor
+       runs at the commanded duty cycle indefinitely in either direction.
+       Using continuous avoids JointSaturationLimiter clamping effort to 0
+       when the joint reaches a revolute position limit. -->
+  <joint name="pwm_joint" type="continuous">
     <parent link="base_link"/>
     <child link="pwm_link"/>
@@ -75,5 +77,6 @@
     <origin xyz="0 0 0.02" rpy="0 0 0"/>
     <axis xyz="0 1 0"/>
-    <limit lower="-3.14159" upper="3.14159" effort="1.0" velocity="5.0"/>
+    <!-- effort limit only (no position limits on continuous joint) -->
+    <limit effort="1.0" velocity="5.0"/>
   </joint>
   <!-- ros2_control hardware interface -->
